File: Hardware/DSP.kicad_sch (KiCad schematic)
At the start: 78 parts, among them IC1 741G17DBV, J1 Conn_02x08_Odd_Even, J10 Conn_01x10_Female, J2 Conn_02x05_Odd_Even, J3 Conn_02x03_Counter_Clockwise, J5 Conn_01x18_Male, J6 Conn_01x10_Male, J7 Conn_01x16_Male, J8 Conn_01x16_Female, J9 Conn_01x18_Female, SW1 SW_SPDT, SW2 SW_SPDT, U1 L7805, U11 NCP1117-3.3_SOT223, U2 NCP1117-3.3_SOT223, U3 6N138, U4 LM4040DBZ-10, U5 L7805, U6 TL072, U7 Teensy4.1, U8 PCM5100, X1 KUSBVX

Commit message: upload everything
Parts:
- removed C14: 100u, Capacitor_SMD:C_Elec_5x5.8, symbol Device:CP
- removed C21, C23: 10u, Capacitor_SMD:C_Elec_5x5.8, symbol Device:CP
- removed C22, C24: 2.2u, Capacitor_SMD:C_Elec_5x5.8, symbol Device:CP
- removed C25, C26, C27, C28, C29: 100n, Capacitor_SMD:C_0805_2012Metric, symbol Device:C
- removed D1, D2: STPS1L30U, Diode_SMD:D_SMB, symbol Device:D_Schottky
- removed J1: Conn_02x08_Odd_Even, con-3m:con-3m-PAK100_2500-16, symbol Connector_Generic:Conn_02x08_Odd_Even
- removed J10: Conn_01x10_Female, Connector_PinSocket_2.54mm:PinSocket_2x05_P2.54mm_Vertical_SMD, symbol Connector:Conn_01x10_Female
- removed J2: Conn_02x05_Odd_Even, Connector_PinHeader_1.27mm:PinHeader_2x05_P1.27mm_Vertical_SMD, symbol Connector_Generic:Conn_02x05_Odd_Even
- removed J3: Conn_02x03_Counter_Clockwise, Connector_PinHeader_2.54mm:PinHeader_2x03_P2.54mm_Vertical_SMD, symbol Connector_Generic:Conn_02x03_Counter_Clockwise
- removed J5: Conn_01x18_Male, Connector_PinHeader_2.54mm:PinHeader_2x09_P2.54mm_Vertical_SMD, symbol Connector:Conn_01x18_Male
- removed J6: Conn_01x10_Male, Connector_PinHeader_2.54mm:PinHeader_2x05_P2.54mm_Vertical_SMD, symbol Connector:Conn_01x10_Male
- removed J7: Conn_01x16_Male, Connector_PinHeader_2.54mm:PinHeader_2x08_P2.54mm_Vertical_SMD, symbol Connector:Conn_01x16_Male
- removed J8: Conn_01x16_Female, Connector_PinSocket_2.54mm:PinSocket_2x08_P2.54mm_Vertical_SMD, symbol Connector:Conn_01x16_Female
- removed J9: Conn_01x18_Female, Connector_PinSocket_2.54mm:PinSocket_2x09_P2.54mm_Vertical_SMD, symbol Connector:Conn_01x18_Female
- removed L1: 33u, Inductor_SMD:L_1206_3216Metric, symbol Device:L
- removed L4, L5: BLM21PG221SN1D, Inductor_SMD:L_0805_2012Metric, symbol Device:L
- removed R10, R39: 10k, Resistor_SMD:R_0805_2012Metric, symbol Device:R
- removed R44, R45: 100k, Resistor_SMD:R_0805_2012Metric, symbol Device:R
- removed SW1, SW2: SW_SPDT, Button_Switch_SMD:SW_SPDT_PCM12, symbol Switch:SW_SPDT
- removed U1, U5: L7805, Package_TO_SOT_SMD:TO-252-2, symbol Regulator_Linear:L7805
- removed U2: NCP1117-3.3_SOT223, Package_TO_SOT_SMD:SOT-223-3_TabPin2, symbol Regulator_Linear:NCP1117-3.3_SOT223
- removed U7: Teensy4.1, teensy:Teensy41-minimal, symbol teensy:Teensy4.1
- removed U8: PCM5100, Package_SO:TSSOP-20_4.4x6.5mm_P0.65mm, symbol Audio:PCM5100
- removed demp1, flt1, fmt1, xsmt1: Jumper_2_Bridged, Jumper:SolderJumper-2_P1.3mm_Open_Pad1.0x1.5mm, symbol Jumper:Jumper_2_Bridged
- added A1: Device_Audio_Electrosmith_Daisy_Seed_Rev4, Device_Audio_Electrosmith_Daisy_Seed:Device_Audio_Electrosmith_Daisy_Seed, symbol Device_Audio_Electrosmith_Daisy_Seed:Device_Audio_Electrosmith_Daisy_Seed_Rev4
- added C14: 470n, Capacitor_SMD:C_0805_2012Metric, symbol Device:C
- added C21, C22: 220u, Capacitor_SMD:CP_Elec_5x5.8, symbol Device:C_Polarized
- added J1: USB_B, Connector_USB:USB_Micro-B_GCT_USB3076-30-A, symbol Connector:USB_B
- added R49, R54: 33k, Resistor_SMD:R_0805_2012Metric, symbol Device:R
- added SW1: SW_SPST, Button_Switch_THT:SW_E-Switch_EG1224_SPDT_Angled, symbol Switch:SW_SPST
- added U2: PESE1-S5-D12-M-TR, vestursynthesis:PESE1, symbol VesturSynthesis:PESE1
- added U5: LM4810, Package_SO:TSSOP-8_3x3mm_P0.65mm, symbol Amplifier_Audio:LM4810
- added d+1, d-1: TestPoint, Connector_Pin:Pin_D1.0mm_L10.0mm, symbol Connector:TestPoint
- added headphone1, line1: AudioJack3, Connector_Audio:Jack_3.5mm_CUI_SJ-3523-SMT_Horizontal, symbol Connector:AudioJack3
- added vol1: R_Potentiometer_Dual, Potentiometer_THT:Potentiometer_Alpha_RD902F-40-00D_Dual_Vertical, symbol Device:R_Potentiometer_Dual
- C18: value 100n -> 470n
- C2: value 100u -> 22u
- L12, L2: value 33u -> 2.2u
- L3: value BLM21PG221SN1D -> 2.2u
- R6: value 10k -> 1k
- R7: value 2.2k -> 1k
- R8: value 2.2k -> 22k
- R9: value 10k -> 22k
- U3: footprint VesturSynthesis:DIL8-SMD -> vestursynthesis:DIL8-SMD
- X1: footprint VesturSynthesis:KUSBVX -> Connector_USB:USB_A_Molex_67643_Horizontal
Connections:
- net 5V_USB is gone; now on net +5V: X1.1
- net D+_F is gone; now on net D+: X1.3
- net D-_F is gone; now on net D-: X1.2
- net RIGHT-OUT is gone; now on an unnamed net: C31.1, U6.7
- net SCL-EXP is gone; now on an unnamed net: R6.2
- net +12V: now also C1.1, U2.5 (-VOUT), U5.8 (VDD); no longer L12.2, L2.2
- net +3.3V: now also A1.38 (3V3_D); no longer C20.1, R6.1
- net +3.3VA: now also A1.21 (3V3_A); no longer C1.1, C2.1
- net +5V: now also L12.2, L2.2, A1.39 (VIN), SW1.2 (B)
- net -12V: now also U2.7 (+VOUT)
- net CONTROL1_CV: now also A1.22 (ADC_INP10)
- net CONTROL2_CV: now also A1.23 (ADC_INP15)
- net D+: now also A1.37 (USB_HS_D_+)
- net D-: now also A1.36 (USB_HS_D_-)
- net GATE: now also A1.10 (SPI1_MISO)
- net GND: now also C1.2, C10.2, C13.2, C15.2, C16.1, C17.2, C19.2, C2.2, C20.2, C3.2, C4.2, C44.2, C5.2, C6.2, C7.1, IC1.3 (GND), R3.1, U11.1 (GND), U3.5 (GND), U4.1 (K), A1.1 (USB_HS_ID), A1.20 (AGND), A1.40 (GND), J1.4 (GND), J1.5 (Shield), U2.1 (GND), U2.4 (0V), U5.4 (GND), U5.5 (SHDN), headphone1.S, vol1.1, vol1.4; no longer C18.2
- net MIDI-RX: now also A1.15 (USART1_RX)
- net SCL: now also A1.12 (I2C1_SCL)
- net SDA: now also A1.13 (I2C1_SDA)
- net ctl1_enc_A: now also A1.3 (SDMMC1_D2)
- net ctl1_enc_B: now also A1.4 (SDMMC1_D1)
- net ctl1_sw: now also A1.11 (SPI1_MOSI)
- net ctl2_enc_A: now also A1.6 (SDMMC1_CMD)
- net ctl2_enc_B: now also A1.5 (SDMMC1_D0)
- net ctl2_sw: now also A1.7 (SDMMC1_CK)
- net dac_left: now also C30.2, U6.3 (+), A1.18 (AUDIO_OUT_L), vol1.6; no longer R7.1
- net dac_right: now also C31.2, U6.5 (+), A1.19 (AUDIO_OUT_R), vol1.3; no longer R8.1
- net midi_sw: now also A1.2 (SDMMC1_D3)
- net switch1_sw: now also A1.8 (SPI1_NSS)
- net switch2_sw: now also A1.9 (SPI1_SCK)
- net at U6.6 (-): now also R7.2; no longer C31.2
- net at L2.1: now also C2.1, U2.2 (VIN)
- net at C18.1: now also vol1.2
- net at R9.1: now also R54.2, U5.6 (VIN2); no longer R7.2
- net at R8.2: now also C14.2
- net at L3.2: now also J1.1 (VBUS)
- removed net GND1: C1.2, C10.2, C13.2, C15.2, C16.1, C17.2, C19.2, C2.2, C20.2, C3.2, C4.2, C44.2, C5.2, C6.2, C7.1, IC1.3 (GND), R3.1, U11.1 (GND), U3.5 (GND), U4.1 (K), U6.3 (+), U6.5 (+)
- net LEFT-OUT: no longer names the net of C30.1, U6.1
- net LEFT-OUT: now also U6.2 (-)
- net euro-5V: no longer names the net of L3.1
- net euro-5V: now also SW1.1 (A)
- new net: R7.1, line1.R
- new net: C20.1, U5.3 (BYPASS)
- new net: C21.1, R49.1, U5.1 (VOUT1)
- new net: R49.2, R8.1, U5.2 (VIN1)
- new net: C22.1, R54.1, U5.7 (VOUT2)
- new net: C22.2, headphone1.R
- new net: J1.2 (D-), d-1.1
- new net: C18.2, R9.2
- new net: R6.1, line1.T
- new net: C21.2, headphone1.T
- new net: J1.3 (D+), d+1.1
- new net: C14.1, vol1.5
- new net A: A1.35 (SAI2_SCK_B)
- new net ATTACK1: A1.27 (ADC_INP11)
- new net ATTACK2: A1.28 (ADC1_INP4)
- new net B: A1.34 (SAI2_FS_B)
- new net C: A1.33 (SAI2_SD_A)
- new net LFO-FREQ: A1.26 (ADC_INP3)
- new net LFO-WAVE: A1.25 (ADC_INP7)
- new net controls: A1.24 (ADC_INP5)
- new net dac1: A1.29 (DAC1_OUT2)
- new net dac2: A1.30 (DAC1_OUT1)
- new net voct: A1.31 (SAI2_MCLK_B)
Other:
- note removed: "IO board"
- note removed: "expander header"
- moved on the sheet: C13, C3, C30, C31, C44, D3, IC1B, L12, R1, R3, R4, R42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
