File: Hardware/DSP.kicad_sch (KiCad schematic)
At the start: 78 parts, among them IC1 741G17DBV, J1 Conn_02x08_Odd_Even, J10 Conn_01x10_Female, J2 Conn_02x05_Odd_Even, J3 Conn_02x03_Counter_Clockwise, J5 Conn_01x18_Male, J6 Conn_01x10_Male, J7 Conn_01x16_Male, J8 Conn_01x16_Female, J9 Conn_01x18_Female, SW1 SW_SPDT, SW2 SW_SPDT, U1 L7805, U11 NCP1117-3.3_SOT223, U2 NCP1117-3.3_SOT223, U3 6N138, U4 LM4040DBZ-10, U5 L7805, U6 TL072, U7 Teensy4.1, U8 PCM5100, X1 KUSBVX

Commit message: update
Parts:
- removed C14: 100u, Capacitor_SMD:C_Elec_5x5.8, symbol Device:CP
- removed C18, C25, C26, C27, C28, C29: 100n, Capacitor_SMD:C_0805_2012Metric, symbol Device:C
- removed C21, C23: 10u, Capacitor_SMD:C_Elec_5x5.8, symbol Device:CP
- removed C22, C24: 2.2u, Capacitor_SMD:C_Elec_5x5.8, symbol Device:CP
- removed J3: Conn_02x03_Counter_Clockwise, Connector_PinHeader_2.54mm:PinHeader_2x03_P2.54mm_Vertical_SMD, symbol Connector_Generic:Conn_02x03_Counter_Clockwise
- removed L3: BLM21PG221SN1D, Inductor_SMD:L_0805_2012Metric, symbol Device:L
- removed R39, R6: 10k, Resistor_SMD:R_0805_2012Metric, symbol Device:R
- removed SW1, SW2: SW_SPDT, Button_Switch_SMD:SW_SPDT_PCM12, symbol Switch:SW_SPDT
- removed U1, U5: L7805, Package_TO_SOT_SMD:TO-252-2, symbol Regulator_Linear:L7805
- removed U7: Teensy4.1, teensy:Teensy41-minimal, symbol teensy:Teensy4.1
- removed U8: PCM5100, Package_SO:TSSOP-20_4.4x6.5mm_P0.65mm, symbol Audio:PCM5100
- removed demp1, flt1, fmt1, xsmt1: Jumper_2_Bridged, Jumper:SolderJumper-2_P1.3mm_Open_Pad1.0x1.5mm, symbol Jumper:Jumper_2_Bridged
- added A1: Device_Audio_Electrosmith_Daisy_Seed_Rev4, Device_Audio_Electrosmith_Daisy_Seed:Device_Audio_Electrosmith_Daisy_Seed, symbol Device_Audio_Electrosmith_Daisy_Seed:Device_Audio_Electrosmith_Daisy_Seed_Rev4
- added C21, C22, C23: 1n, Capacitor_SMD:C_0805_2012Metric, symbol Device:C
- added C24: 100n, Capacitor_SMD:C_0805_2012Metric, symbol Device:C
- added Q2, Q3, Q4, Q5: BC847, Package_TO_SOT_SMD:SOT-23, symbol Device:Q_NPN_BCE
- added R46, R61, R63: 100k 1%, Resistor_SMD:R_0805_2012Metric, symbol Device:R
- added R47, R60, R62: 140k 1%, Resistor_SMD:R_0805_2012Metric, symbol Device:R
- added R48, R49, R58, R59: 10k, Resistor_SMD:R_0805_2012Metric, symbol Device:R
- added R56, R57, R80, R81: 33k 1%, Resistor_SMD:R_0805_2012Metric, symbol Device:R
- added U1: PESE1, vestursynthesis:PESE1, symbol VesturSynthesis:PESE1
- added U7: MCP6004, Package_SO:SOIC-14_3.9x8.7mm_P1.27mm, symbol Amplifier_Operational:MCP6004
- added U8: 74HC4051D, Package_SO:SOIC-16_4.55x10.3mm_P1.27mm, symbol 4xxx:4051
- C20: value 100n -> 1n
- R10: value 10k -> 100k 1%
- R7, R8: value 2.2k -> 47k
- R9: value 10k -> 140k 1%
- X1: footprint VesturSynthesis:KUSBVX -> Connector_USB:USB_A_Molex_67643_Horizontal
Connections:
- net 5V_USB is gone; now on net +5V: X1.1
- net +12V: no longer J2.1 (Pin_1)
- net +3.3V: now also A1.38 (3V3_D), U8.16 (VDD); no longer C20.1, J2.10 (Pin_10)
- net +3.3VA: now also C24.2, U7.4 (V+)
- net +5V: now also A1.39 (VIN), U1.7 (+VOUT)
- net -10V: now also R9.2, R47.2, R60.2, R62.2
- net -12V: no longer J2.9 (Pin_9)
- net ATTACK: now also U8.4 (X7)
- net CONTROL1_CV: now also A1.22 (ADC_INP10)
- net CONTROL2_CV: now also A1.23 (ADC_INP15)
- net CONTROL3: now also U8.13 (X0)
- net D+: now also X1.3, A1.37 (USB_HS_D_+); no longer J9.10 (Pin_10)
- net D-: now also X1.2, A1.36 (USB_HS_D_-); no longer J9.11 (Pin_11)
- net G1-EXP: now also A1.35 (SAI2_SCK_B), Q2.2 (C); no longer J2.2 (Pin_2)
- net G2-EXP: now also A1.34 (SAI2_FS_B), Q3.2 (C); no longer J2.4 (Pin_4)
- net G3-EXP: now also A1.33 (SAI2_SD_A), Q4.2 (C); no longer J2.6 (Pin_6)
- net G4-EXP: now also A1.32 (SAI2_SD_B), Q5.2 (C); no longer J2.8 (Pin_8)
- net GATE: now also A1.10 (SPI1_MISO)
- net GND: no longer X1.4, X1.M1 (S1), X1.M2 (S2)
- net GND1: now also J2.10 (Pin_10), J2.9 (Pin_9), X1.4, X1.M1 (S1), X1.M2 (S2), A1.1 (USB_HS_ID), A1.20 (AGND), A1.40 (GND), C24.1, Q2.3 (E), Q3.3 (E), Q4.3 (E), Q5.3 (E), U1.1 (GND), U1.4 (0V), U7.10 (+), U7.11 (V-), U7.12 (+), U7.3 (+), U7.5 (+), U8.6 (Inh), U8.7 (VEE), U8.8 (VSS); no longer C20.2, J2.7 (Pin_7)
- net MIDI-RX: now also A1.15 (USART1_RX)
- net PM1: now also U8.1 (X4)
- net PM2: now also U8.5 (X5)
- net RATIO1: now also U8.15 (X2)
- net RATIO2: now also U8.12 (X3)
- net RELEASE: now also U8.2 (X6)
- net SCL: now also A1.12 (I2C1_SCL)
- net SDA: now also A1.13 (I2C1_SDA)
- net ctl1_enc_A: now also A1.3 (SDMMC1_D2)
- net ctl1_enc_B: now also A1.4 (SDMMC1_D1)
- net ctl2_enc_A: now also A1.6 (SDMMC1_CMD)
- net ctl2_enc_B: now also A1.5 (SDMMC1_D0)
- net cutoff: now also U8.14 (X1)
- net dac_left: now also A1.18 (AUDIO_OUT_L)
- net dac_right: now also A1.19 (AUDIO_OUT_R)
- net midi_sw: now also A1.2 (SDMMC1_D3)
- net switch1_sw: now also A1.8 (SPI1_NSS)
- net switch2_sw: now also A1.9 (SPI1_SCK)
- net at C31.2, R45.1, U6.6 (-): now also R8.2; no longer R10.2
- net at L1.1: now also U1.2 (VIN)
- net at C30.2, R44.1, U6.2 (-): now also R7.2; no longer R9.2
- net at R9.1: now also R10.1, C21.2, R57.2, U7.6 (-); no longer R7.2
- net at J1.11 (Pin_11): no longer J1.12 (Pin_12)
- net D+_F: no longer names the net of J5.10 (Pin_10)
- net D+_F: no longer X1.3
- net D-_F: no longer names the net of J5.11 (Pin_11)
- net D-_F: no longer X1.2
- net SCL-EXP renamed voct2-I
- net voct2-I: now also R61.2
- net SDA-EXP renamed voct3-I
- net voct3-I: now also R10.2
- net ctl1_sw renamed switch3_sw
- net switch3_sw: now also A1.11 (SPI1_MOSI)
- net ctl1_sw_F renamed switch3_sw_F
- net ctl2_sw renamed switch4_sw
- net switch4_sw: now also A1.7 (SDMMC1_CK)
- net ctl2_sw_F renamed switch4_sw_F
- net sin: no longer names the net of J9.12 (Pin_12)
- net sin-f: no longer names the net of J5.12 (Pin_12)
- new net: Q3.1 (B), R49.2
- new net: Q2.1 (B), R48.2
- new net: C23.2, R62.1, R63.1, R81.2, U7.13 (-)
- new net: Q4.1 (B), R58.2
- new net: C22.2, R60.1, R61.1, R80.2, U7.9 (-)
- new net: Q5.1 (B), R59.2
- new net: C20.2, R46.1, R47.1, R56.2, U7.2 (-)
- new net A: A1.31 (SAI2_MCLK_B), U8.11 (A)
- new net B: A1.30 (DAC1_OUT1), U8.10 (B)
- new net C: A1.29 (DAC1_OUT2), U8.9 (C)
- new net G1-EXP-I: J2.2 (Pin_2), R48.1
- new net G2-EXP-I: J2.4 (Pin_4), R49.1
- new net G3-EXP-I: J2.6 (Pin_6), R58.1
- new net G4-EXP-I: J2.8 (Pin_8), R59.1
- new net controls: A1.24 (ADC_INP5), U8.3 (X)
- new net voct1: A1.28 (ADC1_INP4), C20.1, R56.1, U7.1
- new net voct1-I: J2.1 (Pin_1), R46.2
- new net voct2: A1.27 (ADC_INP11), C22.1, R80.1, U7.8
- new net voct3: A1.26 (ADC_INP3), C21.1, R57.1, U7.7
- new net voct4: A1.25 (ADC_INP7), C23.1, R81.1, U7.14
- new net voct4-I: J2.7 (Pin_7), R63.2
Other:
- note added: "expander"
- note added: "main/DSP board"
- note removed: "IO board"
- moved on the sheet: C10, C13, C17, C44, IC1A, J10, J5, J6, J7, J8, J9, L12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
