File: Hardware/io.kicad_sch (KiCad schematic)
At the start: 126 parts, among them Q1 BC847, SW3 ctl1, SW4 ctl2, U10 MCP6004, U12 PCA9622, U13 MCP6002, U9 MCP6004

Commit message: upload everything
Parts:
- removed C36: 100n, Capacitor_SMD:C_0805_2012Metric, symbol Device:C
- removed L7: BLM21PG221SN1D, Inductor_SMD:L_0805_2012Metric, symbol Device:L
- removed LEFT-OUT1, RIGHT-OUT1: THONKICONNNEW, VesturSynthesis:WQP-PJ301M-12_JACK, symbol VesturSynthesis:THONKICONNNEW
- removed MIDI-IN1, MIDI-THRU1: THONKI-STEREO, VesturSynthesis:WQP-PJ366ST_JACK, symbol VesturSynthesis:THONKI-STEREO
- removed R54: 1k, Resistor_SMD:R_0805_2012Metric, symbol Device:R
- removed U13: MCP6002, Package_SO:SOIC-8-1EP_3.9x4.9mm_P1.27mm_EP2.514x3.2mm, symbol Amplifier_Operational:MCP6002-xMC
- removed sw-midi1: SW_MEC_5G, Button_Switch_THT:SW_TH_Tactile_Omron_B3F-10xx, symbol Switch:SW_MEC_5G
- added ATTACK1, ATTACK2, ENV2-AMP1, LFO-AMP1, LFO-FREQ1, LFO-WAVE1: 50k-lin, VesturSynthesis:9MM_SNAP-IN_POT, symbol Device:R_POT
- added C12, C24: 100n, Capacitor_SMD:C_0805_2012Metric, symbol Device:C
- added C23: 1n, Capacitor_SMD:C_0805_2012Metric, symbol Device:C
- added CV-REL1: THONKICONNNEW, vestursynthesis:WQP-PJ301M-12_JACK, symbol VesturSynthesis:THONKICONNNEW
- added R10, R45, R46: 100k, Resistor_SMD:R_0805_2012Metric, symbol Device:R
- added R39, R44: 200k, Resistor_SMD:R_0805_2012Metric, symbol Device:R
- added R47, R48: 100, Resistor_SMD:R_0805_2012Metric, symbol Device:R
- added R56: 100k 1%, Resistor_SMD:R_0805_2012Metric, symbol Device:R
- added R57: 33k 1%, Resistor_SMD:R_0805_2012Metric, symbol Device:R
- added U13: MCP6001-OT, Package_TO_SOT_SMD:SOT-23-5, symbol Amplifier_Operational:MCP6001-OT
- added U7: MCP6004, Package_SO:SOIC-14_3.9x8.7mm_P1.27mm, symbol Amplifier_Operational:MCP6004
- added U8: 74HC4051D, Package_SO:SOIC-16_4.55x10.3mm_P1.27mm, symbol 4xxx:4051
- added env2-o1, lfo-o1, mult1, mult2, mult3, mult4, pitch1: THONKICONNNEW, VesturSynthesis:WQP-PJ301M-12_JACK, symbol VesturSynthesis:THONKICONNNEW
- added midi-i1, midi-thru1: AudioJack3, Connector_Audio:Jack_3.5mm_CUI_SJ-3523-SMT_Horizontal, symbol Connector:AudioJack3
- added sw-midi1: SW_Push, Button_Switch_THT:SW_Tactile_SKHH_Angled, symbol Switch:SW_Push
- CV-CTL1: renamed from CV-CTL3; footprint VesturSynthesis:WQP-PJ301M-12_JACK -> vestursynthesis:WQP-PJ301M-12_JACK
- CV-CTL2: renamed from CV-CTL4; footprint VesturSynthesis:WQP-PJ301M-12_JACK -> vestursynthesis:WQP-PJ301M-12_JACK
- CV-FILTDEC1: renamed from CV-CTL2; footprint VesturSynthesis:WQP-PJ301M-12_JACK -> vestursynthesis:WQP-PJ301M-12_JACK
- CV-PM2: renamed from CV-PM1; footprint VesturSynthesis:WQP-PJ301M-12_JACK -> vestursynthesis:WQP-PJ301M-12_JACK
- CV-PM3: renamed from CV-PM2; footprint VesturSynthesis:WQP-PJ301M-12_JACK -> vestursynthesis:WQP-PJ301M-12_JACK
- CV-RAT2: renamed from CV-RAT1; footprint VesturSynthesis:WQP-PJ301M-12_JACK -> vestursynthesis:WQP-PJ301M-12_JACK
- CV-RAT3: renamed from CV-RAT2; footprint VesturSynthesis:WQP-PJ301M-12_JACK -> vestursynthesis:WQP-PJ301M-12_JACK
- CV-REL2: renamed from CV-REL1; footprint VesturSynthesis:WQP-PJ301M-12_JACK -> vestursynthesis:WQP-PJ301M-12_JACK
- D4: footprint LED_THT:LED_D3.0mm -> LED_THT:LED_D3.0mm_FlatTop
- R55: value 1k -> 140k 1%
- cv-cutoff1: footprint VesturSynthesis:WQP-PJ301M-12_JACK -> vestursynthesis:WQP-PJ301M-12_JACK
- renumbered cutoff1 to CUTOFF1, CTL2 to FILT-DEC1, PM1 to PM2, PM2 to PM3, RATIO1 to RATIO2, RATIO2 to RATIO3, ATTACK1 to RELEASE1, RELEASE1 to RELEASE2, GATE-OUT1 to gate-o1
Connections:
- net -10V_F is gone; now on net -10V: CUTOFF1.1, FILT-DEC1.1, PM2.1, PM3.1, R66.2, R68.2, RATIO2.1, RATIO3.1, RELEASE1.1, RELEASE2.1
- net led_gate_f is gone; now on net +5V: D4.2 (A)
- net GND: now also ATTACK1.1, ATTACK2.1, C12.1, C24.2, CV-REL1.P$2_SWITCH (SWITCH), CV-REL1.P$3_SLEEVE (SLEEVE), ENV2-AMP1.1, LFO-AMP1.1, LFO-FREQ1.1, LFO-WAVE1.1, R39.2, R44.2, U13.2 (V-), U13.3 (+), U7.11 (V-), U7.3 (+), U7.5 (+), U8.6 (Inh), U8.7 (VEE), U8.8 (VSS), env2-o1.P$3_SLEEVE (SLEEVE), lfo-o1.P$3_SLEEVE (SLEEVE), midi-thru1.S, mult1.P$3_SLEEVE (SLEEVE), mult2.P$3_SLEEVE (SLEEVE), mult3.P$3_SLEEVE (SLEEVE), mult4.P$3_SLEEVE (SLEEVE), pitch1.P$2_SWITCH (SWITCH), pitch1.P$3_SLEEVE (SLEEVE), sw-midi1.2; no longer R5.1
- net at C42.2, R28.1, R29.1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: now also U9.9 (-); no longer U10.9 (-)
- net at C35.2, R17.1, R18.1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: now also U9.13 (-); no longer U9.9 (-)
- net at C32.2, R11.1, R14.1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: now also U10.6 (-); no longer U9.2 (-)
- net at C33.2, R12.1, R13.1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: now also U10.9 (-); no longer U9.13 (-)
- net at C34.2, R15.1, R16.1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: now also U9.2 (-); no longer U9.6 (-)
- net at C41.2, R26.1, R27.1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: now also U9.6 (-); no longer U10.6 (-)
- net at C40.2, R25.1, R32.2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: now also R10.1
- net -10V: now reaches R55.1
- net at C46.2: now also midi-i1.S
- net at L10.2: now also midi-thru1.T
- net at L11.2: now also midi-thru1.R
- net at L8.2: now also midi-i1.T
- net at L9.2: now also midi-i1.R
- net at C9.2, R68.1, R69.1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: now also U7.2 (-)
- net at C8.2, R66.1, R67.1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: now also U7.6 (-)
- net +3.3VA_F renamed +3.3VA
- net +3.3VA: now also ATTACK1.3, ATTACK2.3, C12.2, C24.1, LFO-FREQ1.3, LFO-WAVE1.3, U13.5 (V+), U7.4 (V+)
- net +3.3VP_F renamed +3.3VP
- net +3.3VP: now also R83.2, R84.2, R87.2, R88.2
- removed net +3.3V_F1: R50.2, R83.2, R84.2, R87.2, R88.2
- net 5V_USB renamed +5V
- net ATTACK_F renamed RELEASE1
- net RELEASE1: now also U8.2 (X6)
- net CONTROL1_CV_F renamed CONTROL1_CV
- net CONTROL1_CV: now also U7.1
- net CONTROL2_CV_F renamed CONTROL2_CV
- net CONTROL2_CV: now also U7.7
- net CONTROL3_F renamed CONTROL3
- net CONTROL3: now also U10.8, U8.13 (X0); no longer U9.14
- net GATE-F renamed GATE
- net GATE: now also R5.1
- net MIDI-IN-L-F renamed MIDI-RX5
- net MIDI-IN-R-F renamed MIDI-RX4
- net MIDI-THRU-L-F renamed MIDI-THRU
- net PM1_F renamed PM2
- net PM2: now also U9.7, U8.5 (X5); no longer U10.7
- net PM2_F renamed PM3
- net PM3: now also U9.1, U8.1 (X4); no longer U9.7
- net RATIO1_F renamed RATIO2
- net RATIO2: now also U9.8, U8.15 (X2); no longer U10.8
- net RATIO2_F renamed RATIO3
- net RATIO3: now also U9.14, U8.12 (X3); no longer U9.8
- net RELEASE_F renamed RELEASE2
- net RELEASE2: now also U8.4 (X7)
- net RIGHT-OUT-F: no longer names the net of R55.2
- net RIGHT-OUT-F: now also C23.2, R56.2, R57.1, U13.4 (-)
- net SCL_F renamed SCL
- net SDA_F renamed SDA
- net ctl1_enc_A_F renamed ctl1_enc_A
- net ctl1_enc_B_F renamed ctl1_enc_B
- net ctl1_sw_F renamed ctl1_sw
- net ctl2_enc_A_F renamed ctl2_enc_A
- net ctl2_enc_B_F renamed ctl2_enc_B
- net ctl2_sw_F renamed ctl2_sw
- net cutoff_f renamed cutoff
- net cutoff: now also U10.7, U8.14 (X1); no longer U9.1
- net switch1_sw-F renamed switch1_sw
- net switch2_sw-F renamed switch2_sw
- new net: ENV2-AMP1.3, R46.1, U7.8
- new net: R44.1, R46.2, U7.9 (-)
- new net: R56.1, pitch1.P$1_TIP (TIP)
- new net: LFO-AMP1.3, R45.1, U7.14
- new net: R39.1, R45.2, U7.13 (-)
- new net: R48.1, env2-o1.P$1_TIP (TIP)
- new net: ENV2-AMP1.2, R48.2
- new net: LFO-AMP1.2, R47.2
- new net: mult1.P$1_TIP (TIP), mult2.P$1_TIP (TIP), mult3.P$1_TIP (TIP), mult4.P$1_TIP (TIP)
- new net: R47.1, lfo-o1.P$1_TIP (TIP)
- new net: CV-REL1.P$1_TIP (TIP), R10.2
- new net +3.3V: R50.2, U8.16 (VDD)
- new net A: U8.11 (A)
- new net ATTACK1: ATTACK1.2
- new net ATTACK2: ATTACK2.2
- new net B: U8.10 (B)
- new net C: U8.9 (C)
- new net LFO-FREQ: LFO-FREQ1.2
- new net LFO-WAVE: LFO-WAVE1.2
- new net controls: U8.3 (X)
- new net dac1: U7.10 (+)
- new net dac2: U7.12 (+)
- new net midi_sw: sw-midi1.1
- new net voct: C23.1, R57.2, U13.1
Other:
- moved on the sheet: C11, C37, D4, R5, U10B, U10C, U10E, U9A, U9B, U9C, U9D, U9E
