File: Hardware/io.kicad_sch (KiCad schematic)
At the start: 126 parts, among them Q1 BC847, SW3 ctl1, SW4 ctl2, U10 MCP6004, U12 PCA9622, U13 MCP6002, U9 MCP6004

Commit message: update
Parts:
- sw-midi1, sw-sel1, sw-sel2: footprint Button_Switch_THT:SW_TH_Tactile_Omron_B3F-10xx -> vestursynthesis:SW_TH_Tactile_Omron_B3F-10xx
Connections:
- net ctl1_sw_F is gone; now on net GND: SW3.S2
- net ctl2_sw_F is gone; now on net GND: SW4.S2
- net led_gate_f is gone; now on net euro-5V_f: D4.2 (A)
- net GATE-F: now also R5.1
- net GND: no longer R5.1, SW3.S1, SW4.S1
- net 5V_USB renamed euro-5V_f
- new net switch3_sw_F: SW3.S1
- new net switch4_sw_F: SW4.S1
Other:
- moved on the sheet: C11, C36, C37, D4, L7, R5, U10E, U13C, U9E
